File: wheatstone.kicad_pcb (KiCad board)
At the start: 2 copper layers, 35 x 31 mm, 9 parts, among them J1 Conn_01x03_Pin, J2 Conn_01x02, J3 Conn_01x02

Commit message: final touches
Parts:
- moved Vs1 6.50 mm to (151.0, 95.0)
- moved Vin1 6.00 mm to (137.5, 95.0)
- moved Vp1 3.00 mm to (146.5, 95.0)
- moved GND1 2.50 mm to (142.0, 95.0)
- moved RV1 1.00 mm to (150.5, 88.5)
Routing:
- net +3.3V: track 30.2 -> 33.9 mm
- net Vs: track 29.1 -> 32.4 mm
- net Vp: track 29.7 -> 30.3 mm
Other:
- outline, holes or cut-outs redrawn
Changed lines of the file:
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@@
 		(filling no)
 		(pcbplotparams
-			(layerselection 0x00000000_00000000_55555555_5755f5ff)
+			(layerselection 0x00000000_00000000_55555555_575555ff)
 			(plot_on_all_layers_selection 0x00000000_00000000_00000000_00000000)
 			(disableapertmacros no)
-			(usegerberextensions no)
+			(usegerberextensions yes)
 			(usegerberattributes yes)
 			(usegerberadvancedattributes yes)
@@
 			(outputformat 1)
 			(mirror no)
-			(drillshape 1)
+			(drillshape 0)
 			(scaleselection 1)
-			(outputdirectory "")
+			(outputdirectory "Exports/")
 		)
 	)
 	(footprint "TestPoint:TestPoint_THTPad_D2.5mm_Drill1.2mm"
 		(layer "F.Cu")
-		(at 131.5 95)
+		(at 137.5 95)
 		(descr "THT pad as test Point, diameter 2.5mm, hole diameter 1.2mm ")
 		(tags "test point THT pad")
 		(property "Reference" "Vin1"
-			(at 0 -2.148 0)
+			(at 0 -3 0)
 			(layer "F.SilkS")
 			(effects
@@
 	(footprint "TestPoint:TestPoint_THTPad_D2.5mm_Drill1.2mm"
 		(layer "F.Cu")
-		(at 139.5 95)
+		(at 142 95)
 		(descr "THT pad as test Point, diameter 2.5mm, hole diameter 1.2mm ")
 		(tags "test point THT pad")
 		(property "Reference" "GND1"
-			(at 0 -2.148 0)
+			(at 0 -3 0)
 			(layer "F.SilkS")
 			(effects
@@
 		(tags "Resistor Axial_DIN0207 series Axial Horizontal pin pitch 10.16mm 0.25W = 1/4W length 6.3mm diameter 2.5mm")
 		(property "Reference" "R1"
-			(at 5.08 -2.37 0)
+			(at 5.08 0 0)
 			(layer "F.SilkS")
 			(effects
@@
 	(footprint "TestPoint:TestPoint_THTPad_D2.5mm_Drill1.2mm"
 		(layer "F.Cu")
-		(at 157.5 95)
+		(at 151 95)
 		(descr "THT pad as test Point, diameter 2.5mm, hole diameter 1.2mm ")
 		(tags "test point THT pad")
 		(property "Reference" "Vs1"
-			(at 0 -2.148 0)
+			(at 0 -3 0)
 			(layer "F.SilkS")
 			(effects
@@
 	(footprint "SamacSys_Parts:PV36X101C01B00"
 		(layer "F.Cu")
-		(at 150.46 89.5 -90)
+		(at 150.46 88.5 -90)
 		(descr "PV36X101C01B00-3")
 		(tags "Variable Resistor")
 		(property "Reference" "RV1"
-			(at 0.005 -3.17 90)
+			(at 1 -9.54 0)
 			(layer "F.SilkS")
 			(effects
@@
 		(tags "Connector")
 		(property "Reference" "J2"
-			(at 0 0 90)
+			(at -3.5 2.5 90)
 			(layer "F.SilkS")
 			(effects
@@
 		(tags "Connector")
 		(property "Reference" "J3"
-			(at 0 0 90)
+			(at 3.5 3 90)
 			(layer "F.SilkS")
 			(effects
@@
 	(footprint "TestPoint:TestPoint_THTPad_D2.5mm_Drill1.2mm"
 		(layer "F.Cu")
-		(at 149.5 95)
+		(at 146.5 95)
 		(descr "THT pad as test Point, diameter 2.5mm, hole diameter 1.2mm ")
 		(tags "test point THT pad")
 		(property "Reference" "Vp1"
-			(at 0 -2.148 0)
+			(at 0 -3 0)
 			(layer "F.SilkS")
 			(effects
@@
 		(layer "Edge.Cuts")
 	)
+	(gr_circle
+		(center 130 95)
+		(end 131.5 95)
+		(stroke
+			(width 0.05)
+			(type default)
+		)
+		(fill no)
+		(layer "Edge.Cuts")
+	)
+	(gr_circle
+		(center 140 69)
+		(end 141.5 69)
+		(stroke
+			(width 0.05)
+			(type default)
+		)
+		(fill no)
+		(layer "Edge.Cuts")
+	)
+	(gr_circle
+		(center 149.5 69)
+		(end 151 69)
+		(stroke
+			(width 0.05)
+			(type default)
+		)
+		(fill no)
+		(layer "Edge.Cuts")
+	)
+	(gr_circle
+		(center 159 95)
+		(end 160.5 95)
+		(stroke
+			(width 0.05)
+			(type default)
+		)
+		(fill no)
+		(layer "Edge.Cuts")
+	)
 	(gr_text "Praying\nFor Adiv's\n5k"
 		(at 144.5 78.5 180)
@@
 	)
 	(segment
-		(start 129.92 93.42)
-		(end 131.5 95)
+		(start 137.5 95)
+		(end 135.42 95)
 		(width 0.3)
 		(layer "F.Cu")
@@
 	)
 	(segment
-		(start 129.92 89.5)
-		(end 129.92 93.42)
+		(start 135 77.5)
+		(end 135 78.5)
 		(width 0.3)
 		(layer "F.Cu")
@@
 	)
 	(segment
-		(start 135 77.5)
-		(end 135 78.5)
+		(start 129.92 83.58)
+		(end 129.92 89.5)
 		(width 0.3)
 		(layer "F.Cu")
@@
 	)
 	(segment
-		(start 129.92 83.58)
+		(start 135.42 95)
 		(end 129.92 89.5)
 		(width 0.3)
@@
 	)
 	(segment
-		(start 154 74.5)
-		(end 157.5 78)
+		(start 135 74.5)
+		(end 141.454416 74.5)
 		(width 0.3)
 		(layer "F.Cu")
-		(net "Vs")
+		(net "GND")
 	)
 	(segment
-		(start 153 74.5)
-		(end 152.5 74)
+		(start 141.454416 74.5)
+		(end 141.954416 74)
 		(width 0.3)
 		(layer "F.Cu")
-		(net "Vs")
+		(net "GND")
 	)
 	(segment
-		(start 157.5 78)
-		(end 157.5 95)
+		(start 149.46 89.5)
+		(end 150.46 88.5)
 		(width 0.3)
 		(layer "F.Cu")
-		(net "Vs")
+		(net "Vp")
 	)
 	(segment
-		(start 152.5 74)
-		(end 147.045584 74)
+		(start 150.46 88.5)
+		(end 151 88.5)
 		(width 0.3)
 		(layer "F.Cu")
-		(net "Vs")
+		(net "Vp")
 	)
 	(segment
-		(start 154 74.5)
-		(end 153 74.5)
+		(start 149.46 92.04)
+		(end 149.46 89.5)
 		(width 0.3)
 		(layer "F.Cu")
-		(net "Vs")
+		(net "Vp")
 	)
 	(segment
-		(start 135 74.5)
-		(end 141.454416 74.5)
+		(start 151 88.5)
+		(end 154 85.5)
 		(width 0.3)
 		(layer "F.Cu")
-		(net "GND")
+		(net "Vp")
 	)
 	(segment
-		(start 141.454416 74.5)
-		(end 141.954416 74)
+		(start 154 85.5)
+		(end 154 77.5)
 		(width 0.3)
 		(layer "F.Cu")
-		(net "GND")
+		(net "Vp")
 	)
 	(segment
-		(start 150.46 89.04)
-		(end 154 85.5)
+		(start 140.08 89.5)
+		(end 149.46 89.5)
 		(width 0.3)
 		(layer "F.Cu")
@@
 	)
 	(segment
-		(start 150.46 89.5)
-		(end 150.46 89.04)
+		(start 146.5 95)
+		(end 149.46 92.04)
 		(width 0.3)
 		(layer "F.Cu")
@@
 	)
 	(segment
-		(start 150.46 94.04)
-		(end 149.5 95)
+		(start 153 74.5)
+		(end 152.5 74)
 		(width 0.3)
 		(layer "F.Cu")
-		(net "Vp")
+		(net "Vs")
 	)
 	(segment
-		(start 154 85.5)
-		(end 154 77.5)
+		(start 154 74.5)
+		(end 157.5 78)
 		(width 0.3)
 		(layer "F.Cu")
-		(net "Vp")
+		(net "Vs")
 	)
 	(segment
-		(start 150.46 89.5)
-		(end 150.46 94.04)
+		(start 152.5 74)
+		(end 147.045584 74)
 		(width 0.3)
 		(layer "F.Cu")
-		(net "Vp")
+		(net "Vs")
 	)
 	(segment
-		(start 140.08 89.5)
-		(end 150.46 89.5)
+		(start 154 74.5)
+		(end 153 74.5)
 		(width 0.3)
 		(layer "F.Cu")
-		(net "Vp")
+		(net "Vs")
+	)
+	(segment
+		(start 157.5 78)
+		(end 157.5 89.5)
+		(width 0.3)
+		(layer "F.Cu")
+		(net "Vs")
+	)
+	(segment
+		(start 157.5 89.5)
+		(end 152 95)
+		(width 0.3)
+		(layer "F.Cu")
+		(net "Vs")
+	)
+	(segment
+		(start 152 95)
+		(end 151 95)
+		(width 0.3)
+		(layer "F.Cu")
+		(net "Vs")
 	)
 	(zone
